Commit message: Enabling vision pipeline

File: src/bluerov_sim/urdf/bluerov2.urdf (robot description, URDF)
Before this commit: robot bluerov2, 12 links, 11 joints
Links:
- added link dropper_link, mass 0.001
- added link torpedo_shooter_left_link, mass 0.001
- added link torpedo_shooter_right_link, mass 0.001
Joints:
- added joint dropper_joint: type fixed, parent base_link, child dropper_link, origin xyz=0.0 0.0 -0.08 rpy=0 0 0
- added joint torpedo_shooter_left_joint: type fixed, parent base_link, child torpedo_shooter_left_link, origin xyz=0.20 0.05 0.0 rpy=0 0 0
- added joint torpedo_shooter_right_joint: type fixed, parent base_link, child torpedo_shooter_right_link, origin xyz=0.20 -0.05 0.0 rpy=0 0 0
